File: Hackpad/Hackpad.kicad_sch (KiCad schematic)
At the start: 8 parts, among them SW1 SW_Push_45deg, SW2 SW_Push_45deg, SW3 SW_Push_45deg, SW4 SW_Push_45deg, SW5 RotaryEncoder_Switch_MP, U1 XIAO-RP2040-DIP

Commit message: Resubmission
Parts:
- added D3, D4: SK6805, LED_SMD:LED_SK6805_PLCC4_2.4x2.7mm_P1.3mm, symbol LED:SK6805
- added SW6, SW7, SW8: SW_Push_45deg, PCM_Switch_Keyboard_Cherry_MX:SW_Cherry_MX_PCB_1.00u, symbol Switch:SW_Push_45deg
- U1: footprint Module:MOUDLE14P-XIAO-DIP-SMD -> Seeed Studio XIAO Series Library:XIAO-RP2040-SMD
Connections:
- net +5V: now also D3.4 (VDD), D4.4 (VDD)
- net GND: now also D3.2 (VSS), D4.2 (VSS), SW6.1, SW7.1, SW8.1
- net at U1.6 (GPIO7/SCL): now also SW6.2
- net at U1.7 (GPIO0/TX): now also SW7.2
- net at U1.8 (GPIO1/RX): now also SW8.2
- net at D2.1 (DOUT): now also D3.3 (DIN)
- new net: D3.1 (DOUT), D4.3 (DIN)
Other:
- moved on the sheet: SW1, SW2, SW3, SW4
